File: hardware/pcb-controller/dyad-controller.kicad_sch (KiCad schematic)
At the start: 36 parts, among them J1 USB_C_Receptacle_USB2.0, J2 SWD, J3 Conn_01x11, J4 Conn_01x11, J5 Conn_01x11, SW1 SW_Push, U1 W25Q128JVS, U2 USBLC6-2SC6, U3 RP2040, U4 XC6206PxxxMR-Regulator_Linear, Y1 12MHz

Commit message: Fix controller DRC/ERC and upgrade the schematic to the KiCad 10 format
Most of this diff is mechanical. KiCad rewrote the schematic from format
20211123 (KiCad 6, inherited from the vendored RP2040-designguide) to
20260306, and the board's zone fill was recomputed and its segment list
reordered. The substantive changes are small and listed below.

Schematic:
- #PWR024 was a "+3.3V" power symbol while the rest of the board uses
  "+3V3". KiCad treats those as two separate rails, so U4's regulator
  output and its 1uF cap C17 were isolated from everything they power.
  Renamed to +3V3; the LDO output now actually reaches the RP2040's
  IOVDD/USB_VDD/VREG_VIN pins and the flash.
- Added PWR_FLAGs on GND, +5V and VBUS. ERC errors 4 -> 1.
- U4 repointed from the missing kicad-keyboard-parts library to
  Regulator_Linear:XC6206PxxxMR -- same pin numbers, names, coordinates
  and nets, so nothing moved.

Board:
- U3 and J1 were marked (attr smd) but carry through-hole pads (U3's
  thermal-pad stitching vias, J1's shield tabs). Set to through_hole.
  Note: do not export position files with --smd-only now, or the RP2040
  drops out of the CPL.
- GND zone clearance 0.3 -> 0.15 mm and board min_clearance 0.2 -> 0.15,
  matching JLCPCB's limit. At 0.3 mm the pour retracted far enough to
  isolate a GND pad; the relaxation avoids that, at the cost of one
  extra starved-thermal warning that the next change then clears.
- Five GND pads (U3 x2, U2, Y1, J2) set to solid zone connection instead
  of thermal relief. Thermal relief exists to ease hand-soldering and
  buys nothing on a reflowed ground pad, while hurting the RP2040's heat
  path to the plane.
- Zones refilled and saved so the stored fill matches the board's rules.
  The stale fill was what produced the original clearance violations.

Libraries:
- Registered Sleep-Lib in fp-lib-table. The tables were copied verbatim
  from upstream, which registers the nickname "Footprints", while this
  board references "Sleep-Lib".
- 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
Parts:
- R2: value (none) -> 1k; footprint (none) -> Resistor_SMD:R_0402_1005Metric
- U4: symbol kicad-keyboard-parts:XC6206PxxxMR-Regulator_Linear -> Regulator_Linear:XC6206PxxxMR
