File: hardware/pcb-main-left/dyad-main-left.kicad_pcb (KiCad board)
At the start: 2 copper layers, 149 x 120.7 mm, 129 parts, among them SW1 SW_Push, SW10 SW_Push, SW11 SW_Push, SW12 SW_Push, SW13 SW_Push, SW14 SW_Push, SW15 SW_Push, SW16 SW_Push, SW17 SW_Push, SW18 SW_Push, SW19 SW_Push, SW2 SW_Push, SW20 SW_Push, SW21 SW_Push, SW22 SW_Push, SW23 SW_Push, SW24 SW_Push, SW25 SW_Push, SW26 SW_Push, SW27 SW_Push, SW28 SW_Push, SW29 SW_Push, SW3 SW_Push, SW30 SW_Push, SW31 SW_Push, SW32 SW_Push, SW4 SW_Push, SW5 SW_Push, SW6 SW_Push, SW7 SW_Push, SW8 SW_Push, SW9 SW_Push

Commit message: Left half fully routed, and repair a dragged board-outline corner
330 segments and 32 vias close every connection on main-left. Unconnected
125 -> 0, schematic parity 98 -> 0, no shorts.

Routing also caught a board-outline break that DRC reported as three
invalid_outline errors -- "Board has malformed outline (not a closed shape)".
Nothing was deleted: a three-segment rounded corner had been dragged by
exactly (-6.137, -4.900) mm, leaving a 2.85 mm gap where it belonged and a
dangling spur where it landed. Segment count stayed at 23 either way, which
is why it was not obvious; the tell was four Edge.Cuts endpoints used once
instead of zero.

Restored the three segments to their committed coordinates, then refilled
both pours -- they had been filled against the displaced edge and sat at
0.0000 mm from the restored one, which surfaced as two copper_edge_clearance
errors in between.

  invalid_outline        3 -> 0
  copper_edge_clearance  0 -> 2 -> 0
  Edge.Cuts open ends    4 -> 0

Both halves now carry only cosmetic silkscreen warnings and the deliberate
D/SW courtyard overlaps:

              violations  errors  unconnected  parity  shorts
  main-left          195      32            0       0       0
  main-right         253      37            0       0       0

Co-Authored-By: Claude Opus 5 <noreply@anthropic.com>
Parts:
- moved C28 8.16 mm to (56.0, 117.2), turned to 90 degrees
- moved C27 8.16 mm to (37.0, 117.2), turned to 90 degrees
- moved C29 8.16 mm to (77.5, 117.2), turned to 90 degrees
- moved C30 8.16 mm to (101.3, 117.2), turned to 90 degrees
- moved C31 8.12 mm to (125.0, 117.5), turned to 75 degrees
- moved C15 8.11 mm to (39.3, 79.3), turned to 90 degrees
- moved C16 8.11 mm to (65.5, 79.3), turned to 90 degrees
- moved C17 8.11 mm to (84.5, 79.3), turned to 90 degrees
- moved C18 8.11 mm to (103.6, 79.3), turned to 90 degrees
- moved C19 8.11 mm to (122.7, 79.3), turned to 90 degrees
- moved C20 8.11 mm to (141.7, 79.3), turned to 90 degrees
- moved C3 8.02 mm to (70.3, 41.3), turned to 90 degrees
- moved C4 8.02 mm to (89.3, 41.3), turned to 90 degrees
- moved C7 8.02 mm to (146.5, 41.3), turned to 90 degrees
- moved C1 8.02 mm to (32.2, 41.3), turned to 90 degrees
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Connections:
- LED1 pad 2: LEDIN -> Net-(LED1-DIN)
- LED15 pad 2: Net-(LED14-DOUT) -> Net-(LED15-DIN)
- LED16 pad 2: Net-(LED15-DOUT) -> Net-(LED16-DIN)
- LED16 pad 4: Net-(LED16-DOUT) -> Net-(LED15-DIN)
- LED17 pad 2: Net-(LED16-DOUT) -> Net-(LED17-DIN)
- LED17 pad 4: Net-(LED17-DOUT) -> Net-(LED16-DIN)
- LED18 pad 2: Net-(LED17-DOUT) -> Net-(LED18-DIN)
- LED18 pad 4: Net-(LED18-DOUT) -> Net-(LED17-DIN)
- LED19 pad 2: Net-(LED18-DOUT) -> Net-(LED19-DIN)
- LED19 pad 4: Net-(LED19-DOUT) -> Net-(LED18-DIN)
- LED2 pad 2: Net-(LED1-DOUT) -> Net-(LED2-DIN)
- LED2 pad 4: Net-(LED2-DOUT) -> Net-(LED1-DIN)
- LED20 pad 2: Net-(LED19-DOUT) -> Net-(LED14-DOUT)
- LED20 pad 4: Net-(LED20-DOUT) -> Net-(LED19-DIN)
- LED21 pad 2: Net-(LED20-DOUT) -> Net-(LED15-DOUT)
- LED27 pad 2: Net-(LED26-DOUT) -> Net-(LED27-DIN)
- LED27 pad 4: Net-(LED27-DOUT) -> LEDOUT
- LED28 pad 2: Net-(LED27-DOUT) -> Net-(LED28-DIN)
- LED28 pad 4: Net-(LED28-DOUT) -> Net-(LED27-DIN)
- LED29 pad 2: Net-(LED28-DOUT) -> Net-(LED29-DIN)
- LED29 pad 4: Net-(LED29-DOUT) -> Net-(LED28-DIN)
- LED3 pad 2: Net-(LED2-DOUT) -> Net-(LED3-DIN)
- LED3 pad 4: Net-(LED3-DOUT) -> Net-(LED2-DIN)
- LED30 pad 2: Net-(LED29-DOUT) -> Net-(LED30-DIN)
- LED30 pad 4: Net-(LED30-DOUT) -> Net-(LED29-DIN)
- LED31 pad 2: Net-(LED30-DOUT) -> Net-(LED31-DIN)
- LED31 pad 4: Net-(LED31-DOUT) -> Net-(LED30-DIN)
- LED32 pad 2: Net-(LED31-DOUT) -> Net-(LED26-DOUT)
- LED32 pad 4: LEDOUT -> Net-(LED31-DIN)
- LED4 pad 2: Net-(LED3-DOUT) -> Net-(LED4-DIN)
- LED4 pad 4: Net-(LED4-DOUT) -> Net-(LED3-DIN)
- LED5 pad 2: Net-(LED4-DOUT) -> Net-(LED5-DIN)
- LED5 pad 4: Net-(LED5-DOUT) -> Net-(LED4-DIN)
- LED6 pad 2: Net-(LED5-DOUT) -> Net-(LED6-DIN)
- LED6 pad 4: Net-(LED6-DOUT) -> Net-(LED5-DIN)
- LED7 pad 2: Net-(LED6-DOUT) -> LEDIN
- LED7 pad 4: Net-(LED7-DOUT) -> Net-(LED6-DIN)
- LED8 pad 2: Net-(LED7-DOUT) -> Net-(LED1-DOUT)
Routing:
- net ROW1: track 0.00 -> 120.7 mm
- net ROW0: track 0.00 -> 115.9 mm
- net VCC: track 0.00 -> 110.3 mm, vias 0 -> 32
- net ROW3: track 0.00 -> 109.9 mm
- net ROW4: track 0.00 -> 108.0 mm
- net ROW2: track 0.00 -> 103.9 mm
- net COL5: track 67.0 -> 103.7 mm
- net Net-(LED26-DOUT): track 0.00 -> 29.2 mm
- net Net-(LED31-DIN): track 0.00 -> 29.1 mm
- net COL1: track 67.0 -> 94.5 mm
- net COL2: track 67.0 -> 94.3 mm
- net Net-(LED21-DOUT): track 0.00 -> 26.1 mm
- net Net-(LED14-DOUT): track 0.00 -> 25.8 mm
- net COL4: track 67.0 -> 89.7 mm
- net Net-(LED1-DOUT): track 0.00 -> 22.2 mm
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