File: hardware/pcb-main-right/dyad-main-right.kicad_pcb (KiCad board)
At the start: 2 copper layers, 167.2 x 120.7 mm, 149 parts, among them J1 HC-FPC-0.5-20P-FH20, SW1 SW_Push, SW10 SW_Push, SW11 SW_Push, SW12 SW_Push, SW13 SW_Push, SW14 SW_Push, SW15 SW_Push, SW16 SW_Push, SW17 SW_Push, SW18 SW_Push, SW19 SW_Push, SW2 SW_Push, SW20 SW_Push, SW21 SW_Push, SW22 SW_Push, SW23 SW_Push, SW24 SW_Push, SW25 SW_Push, SW26 SW_Push, SW27 SW_Push, SW28 SW_Push, SW29 SW_Push, SW3 SW_Push, SW30 SW_Push, SW31 SW_Push, SW32 SW_Push, SW33 SW_Push, SW34 SW_Push, SW35 SW_Push, SW36 SW_Push, SW37 SW_Push, SW4 SW_Push, SW5 SW_Push, SW6 SW_Push, SW7 SW_Push, SW8 SW_Push, SW9 SW_Push

Commit message: Delete the dangling ROW4 stub left by the reroute
Two F.Cu segments, not one: the 0.063 mm fragment DRC reported at
(61.28, 114.16) and the diagonal feeding it back to the via at
(61.60, 113.84). Both hung off that via with nothing at the far end; the
via's real connection northward is untouched, and unconnected stays 0.

DRC violations 254 -> 253, which is the pre-connector baseline exactly. The
remaining 253 are the documented ones: 37 courtyards_overlap from the
deliberate diode-under-switch placement, and 216 silkscreen findings.

The one schematic_parity issue is unrelated and still expected -- J1's
Pinout field text, schematic ahead of board, clearing on the next Update PCB
from Schematic.

Co-Authored-By: Claude Opus 5 <noreply@anthropic.com>
Routing:
- net ROW4: track 188.3 -> 187.8 mm
Changed lines of the file:
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@@
-	(segment
-		(start 61.595421 113.841523)
-		(end 61.281528 114.155416)
-		(width 0.2)
-		(layer "F.Cu")
-		(net "ROW4")
-	)
 	(segment
 		(start 61.595421 113.841523)
@@
 		(width 0.2)
 		(layer "F.Cu")
-		(net "ROW4")
-	)
-	(segment
-		(start 61.281528 114.155416)
-		(end 61.281528 114.218472)
-		(width 0.2)
-		(layer "F.Cu")
